File: hid-controller-pcb/hid-controller-pcb.kicad_sch (KiCad schematic)
At the start: 39 parts, among them IC1 RT9080-33GJ5, J1 10118194-0011LF, J2 Jumper, U1 STM32F103C8Tx, U2 32.768KHz, U3 COM-09032, U4 COM-09032, Y1 8MHz

Commit message: schematic finished? now onto layout
Parts:
- removed D1: 3.3V, symbol Device:D_TVS_Small
- added C6, C7: 0.1uF, Capacitor_SMD:C_0603_1608Metric, symbol Device:C_Small
- added C8: 2.2uF, Capacitor_SMD:C_0603_1608Metric, symbol Device:C_Small
- added D1: 3.4V, lib:SMFA2005CA, symbol lib:SMF3.3
- added D2: 6V, lib:DIODE_VESD05A1B-HD1-GS08_VIS, symbol lib:VESD05A1B-HD1-GS08
- C1: footprint (none) -> Capacitor_SMD:C_0603_1608Metric
- C2, C3: value 30pF -> 26pF; footprint (none) -> Capacitor_SMD:C_0603_1608Metric
- C4, C5: value 13pF -> 8pF; footprint (none) -> Capacitor_SMD:C_0603_1608Metric
- J2: footprint (none) -> Connector_PinHeader_2.54mm:PinHeader_1x03_P2.54mm_Vertical
- R1, R10, R11, R12, R13, R14, R15, R16, R2, R3, R4, R5, R6, R7, R8, R9: footprint (none) -> Resistor_SMD:R_0603_1608Metric
Connections:
- net +3V3: now also C7.1, C8.1, D1.1 (K)
- net +5V: now also C1.1, C6.1, D2.1; no longer C1.2
- net BTN_1: now also U1.42 (PB6)
- net BTN_2: now also U1.43 (PB7)
- net BTN_3: now also U1.45 (PB8)
- net BTN_4: now also U1.46 (PB9)
- net DPAD_1: now also U1.16 (PA6)
- net DPAD_2: now also U1.17 (PA7)
- net DPAD_3: now also U1.29 (PA8)
- net DPAD_4: now also U1.30 (PA9)
- net GND: now also C1.2, C6.2, C7.2, C8.2, D1.2 (A), D2.2; no longer C1.1
- net SWDIO: now reaches U1.34 (PA13)
- net SWCLK: now reaches U1.37 (PA14)
Other:
- note added: "ESD PROTECTION"
- moved on the sheet: R10, R11, R12, R13, R14, R15, R16, R9, S1, S2, S3, S4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

Commit message: gruelling layout work on the LSE / HSE oscillators
Parts:
- removed C1: 4.7uF, Capacitor_SMD:C_0603_1608Metric, symbol Device:C_Small
- removed C8: 2.2uF, Capacitor_SMD:C_0603_1608Metric, symbol Device:C_Small
- removed U2: 32.768KHz, lib:CM200C32768DZCT, symbol library:CM200C32768DZCT
- added C1, C8: 10uF, lib:CAPAE530X550N, symbol Device:C_Polarized_Small
- added R17, R19: 0R, Resistor_SMD:R_0603_1608Metric, symbol Device:R_Small
- added R18: 663R, Resistor_SMD:R_0603_1608Metric, symbol Device:R_Small
- added Y2: 32.768KHz, lib:XTAL_ABS25-32.768KHZ-6-T, symbol lib:ABS25-32.768KHZ-6-T
- C2, C3: value 26pF -> 30pF
- C4, C5: value 8pF -> 6pF
Connections:
- net +3V3: now also C8.1
- net +5V: now also C1.1
- net GND: now also C1.2, C8.2, R19.1; no longer U1.20 (PB2)
- net OSC32_IN: now also Y2.1
- net OSC32_OUT: now also R17.2; no longer C5.2
- net OSC_OUT: now also R18.2; no longer C3.2, Y1.1
- new net: C5.2, R17.1, Y2.4
- new net: C3.2, R18.1, Y1.1
- new net BOOT1: R19.2, U1.20 (PB2)
Other:
- moved on the sheet: C6, C7, D1, D2

Commit message: working ADC reading, troubleshooting USB enumeration issues on pc
Parts:
- added C10, C11, C9: 10uF, lib:CAPAE530X550N, symbol Device:C_Polarized_Small
- added C12, C13, C14: 0.1uF, Capacitor_SMD:C_0603_1608Metric, symbol Device:C_Small
Connections:
- net +3V3: now also U1.1 (VBAT), U1.24 (VDD), U1.36 (VDD), U1.48 (VDD), U1.9 (VDDA), C10.1, C11.1, C12.1, C13.1, C14.1, C9.1
- net GND: now also C10.2, C11.2, C12.2, C13.2, C14.2, C9.2
- no-connect marks 1 -> 0
Other:
- note added: "ESD PROTECTION + DECOUPLING CAP"
- note removed: "ESD PROTECTION"
- moved on the sheet: C1, C6, C7, C8, D1, D2
